File: pcb/stm32f091.sch (KiCad schematic (older format))
At the start: 33 parts, among them J3 Conn_02x05_Odd_Even, J4 Conn_02x03_Odd_Even, J5 Conn_02x03_Odd_Even, SW1 SW_Push, U1 LD1117S33TR_SOT223, U2 STM32F091RCTx, X1 32.768kHz(12.5pF), X2 8MHz(20pF)

Commit message: schematic work
Connections:
- net labels removed: PA0, PA1, PA10, PA11, PA12, PA15, PA2, PA3, PA5, PA6, PA7, PA8, PA9, PB0, PB1, PB10, PB11, PB12, PB13, PB15, PB2, PB4, PB8, PB9, PC0, PC1, PC10, PC11, PC12, PC13, PC2, PC3, PC4, PC5, PC6, PC7, PC8, PC9
- wire segments 137 -> 97
Changed lines of the file:
@@
 encoding utf-8
 Sheet 1 1
-Title "STM32F091 Dev Board"
-Date "2020-06-22"
+Title "Group 28"
+Date "2021-11-30"
 Rev "1"
 Comp ""
@@
 Wire Wire Line
 	2650 3250 2850 3250
-$Comp
-L MCU_ST_STM32F0:STM32F091RCTx U2
-U 1 1 5EE02F8A
-P 6200 3100
-F 0 "U2" H 5450 4200 50  0000 C CNN
-F 1 "STM32F091RCTx" H 6050 4200 50  0000 C CNN
-F 2 "Package_QFP:LQFP-64_10x10mm_P0.5mm" H 5600 1400 50  0001 R CNN
-F 3 "http://www.st.com/st-web-ui/static/active/en/resource/technical/document/datasheet/DM00115237.pdf" H 6200 3100 50  0001 C CNN
-	1    6200 3100
-	1    0    0    -1
-$EndComp
-Wire Wire Line
-	6800 1500 7250 1500
-Wire Wire Line
-	6800 1600 7250 1600
-Wire Wire Line
-	6800 1700 7250 1700
-Wire Wire Line
-	6800 1800 7250 1800
 Wire Wire Line
 	6800 1900 7250 1900
 Wire Wire Line
-	6800 2000 7250 2000
-Wire Wire Line
-	6800 2100 7250 2100
-Wire Wire Line
-	6800 2200 7250 2200
-Wire Wire Line
-	6800 2300 7250 2300
-Wire Wire Line
-	6800 2400 7250 2400
-Wire Wire Line
-	6800 2500 7250 2500
-Wire Wire Line
-	6800 2600 7250 2600
-Wire Wire Line
-	6800 2700 7250 2700
-Wire Wire Line
 	6800 2800 7250 2800
 Wire Wire Line
 	6800 2900 7250 2900
 Wire Wire Line
-	6800 3000 7250 3000
-Wire Wire Line
-	6800 3200 7250 3200
-Wire Wire Line
-	6800 3300 7250 3300
-Wire Wire Line
-	6800 3400 7250 3400
-Wire Wire Line
-	6800 3500 7250 3500
-Wire Wire Line
-	6800 3600 7250 3600
-Wire Wire Line
 	6800 3700 7250 3700
 Wire Wire Line
-	6800 3800 7250 3800
-Wire Wire Line
 	6800 3900 7250 3900
 Wire Wire Line
-	6800 4000 7250 4000
-Wire Wire Line
-	6800 4100 7250 4100
-Wire Wire Line
-	6800 4200 7250 4200
-Wire Wire Line
-	6800 4300 7250 4300
-Wire Wire Line
-	6800 4400 7250 4400
-Wire Wire Line
-	6800 4500 7250 4500
-Wire Wire Line
 	6800 4600 7250 4600
 Wire Wire Line
-	6800 4700 7250 4700
-Wire Wire Line
 	5500 2600 5050 2600
 Wire Wire Line
@@
 	5500 3000 5050 3000
 Wire Wire Line
-	5500 3200 5050 3200
-Wire Wire Line
-	5500 3300 5050 3300
-Wire Wire Line
-	5500 3400 5050 3400
-Wire Wire Line
-	5500 3500 5050 3500
-Wire Wire Line
-	5500 3600 5050 3600
-Wire Wire Line
-	5500 3700 5050 3700
-Wire Wire Line
-	5500 3800 5050 3800
-Wire Wire Line
-	5500 3900 5050 3900
-Wire Wire Line
-	5500 4000 5050 4000
-Wire Wire Line
-	5500 4100 5050 4100
-Wire Wire Line
-	5500 4200 5050 4200
-Wire Wire Line
-	5500 4300 5050 4300
-Wire Wire Line
-	5500 4400 5050 4400
-Wire Wire Line
-	5500 4500 5050 4500
-Wire Wire Line
-	5500 4600 5050 4600
-Wire Wire Line
-	5500 4700 5050 4700
-Wire Wire Line
 	5500 1500 5050 1500
-Text Label 7050 1500 0    50   ~ 0
-PA0
-Text Label 7050 1600 0    50   ~ 0
-PA1
-Text Label 7050 1700 0    50   ~ 0
-PA2
-Text Label 7050 1800 0    50   ~ 0
-PA3
 Text Label 7050 1900 0    50   ~ 0
 PA4
-Text Label 7050 2000 0    50   ~ 0
-PA5
-Text Label 7050 2100 0    50   ~ 0
-PA6
-Text Label 7050 2200 0    50   ~ 0
-PA7
-Text Label 7050 2300 0    50   ~ 0
-PA8
-Text Label 7050 2400 0    50   ~ 0
-PA9
-Text Label 7050 2500 0    50   ~ 0
-PA10
-Text Label 7050 2600 0    50   ~ 0
-PA11
-Text Label 7050 2700 0    50   ~ 0
-PA12
 Text Label 7050 2800 0    50   ~ 0
 PA13
 Text Label 7050 2900 0    50   ~ 0
 PA14
-Text Label 7050 3000 0    50   ~ 0
-PA15
-Text Label 7050 3200 0    50   ~ 0
-PB0
-Text Label 7050 3300 0    50   ~ 0
-PB1
-Text Label 7050 3400 0    50   ~ 0
-PB2
-Text Label 7050 3500 0    50   ~ 0
-PB3
-Text Label 7050 3600 0    50   ~ 0
-PB4
-Text Label 7050 3700 0    50   ~ 0
-PB5
-Text Label 7050 3800 0    50   ~ 0
-PB6
 Text Label 7050 3900 0    50   ~ 0
 PB7
-Text Label 7050 4000 0    50   ~ 0
-PB8
-Text Label 7050 4100 0    50   ~ 0
-PB9
-Text Label 7050 4200 0    50   ~ 0
-PB10
-Text Label 7050 4300 0    50   ~ 0
-PB11
-Text Label 7050 4400 0    50   ~ 0
-PB12
-Text Label 7050 4500 0    50   ~ 0
-PB13
 Text Label 7050 4600 0    50   ~ 0
 PB14
-Text Label 7050 4700 0    50   ~ 0
-PB15
-Text Label 5150 3200 0    50   ~ 0
-PC0
-Text Label 5150 3300 0    50   ~ 0
-PC1
-Text Label 5150 3400 0    50   ~ 0
-PC2
-Text Label 5150 3500 0    50   ~ 0
-PC3
-Text Label 5150 3600 0    50   ~ 0
-PC4
-Text Label 5150 3700 0    50   ~ 0
-PC5
-Text Label 5150 3800 0    50   ~ 0
-PC6
-Text Label 5150 3900 0    50   ~ 0
-PC7
-Text Label 5150 4000 0    50   ~ 0
-PC8
-Text Label 5150 4100 0    50   ~ 0
-PC9
-Text Label 5150 4200 0    50   ~ 0
-PC10
-Text Label 5150 4300 0    50   ~ 0
-PC11
-Text Label 5150 4400 0    50   ~ 0
-PC12
-Text Label 5150 4500 0    50   ~ 0
-PC13
-Text Label 5150 4600 0    50   ~ 0
-PC14
-Text Label 5150 4700 0    50   ~ 0
-PC15
 Text Label 5150 2600 0    50   ~ 0
 PF0
@@
 Wire Wire Line
 	6300 1300 6300 1000
-Wire Wire Line
-	5900 4900 6000 4900
-Wire Wire Line
-	6000 4900 6100 4900
-Connection ~ 6000 4900
-Wire Wire Line
-	6100 4900 6200 4900
 Connection ~ 6100 4900
-Wire Wire Line
-	6200 4900 6300 4900
-Connection ~ 6200 4900
 $Comp
 L power:GND #PWR0114
@@
 Wire Notes Line
 	9250 600  9250 6450
+Connection ~ 6200 4900
+Wire Wire Line
+	6200 4900 6300 4900
+Wire Wire Line
+	6100 4900 6200 4900
+Connection ~ 6000 4900
+Wire Wire Line
+	6000 4900 6100 4900
+Wire Wire Line
+	5900 4900 6000 4900
+$Comp
+L MCU_ST_STM32F0:STM32F091RCTx U2
+U 1 1 5EE02F8A
+P 6200 3100
+F 0 "U2" H 5450 4200 50  0000 C CNN
+F 1 "STM32F091RCTx" H 6050 4200 50  0000 C CNN
+F 2 "Package_QFP:LQFP-64_10x10mm_P0.5mm" H 5600 1400 50  0001 R CNN
+F 3 "http://www.st.com/st-web-ui/static/active/en/resource/technical/document/datasheet/DM00115237.pdf" H 6200 3100 50  0001 C CNN
+	1    6200 3100
+	1    0    0    -1
+$EndComp
+Text Label 7050 3700 0    50   ~ 0
+PB5
+Text Label 7050 3500 0    50   ~ 0
+PB3
+Wire Wire Line
+	6800 3500 7250 3500
+Text Label 7050 3800 0    50   ~ 0
+PB6
+Wire Wire Line
+	6800 3800 7250 3800
 $EndSCHEMATC

Commit message: schematic complete
Parts:
- removed J4, J5: Conn_02x03_Odd_Even, Connector_PinHeader_1.27mm:PinHeader_2x03_P1.27mm_Vertical, symbol Connector_Generic:Conn_02x03_Odd_Even
- added C10: 1uF, Capacitor_SMD:C_0805_2012Metric_Pad1.15x1.40mm_HandSolder, symbol Device:C_Small
- added C16, C17, C18, C19: 10uF, Capacitor_SMD:C_0805_2012Metric_Pad1.15x1.40mm_HandSolder, symbol Device:C_Small
- added C20, C21: 0.1uF, Capacitor_SMD:C_0805_2012Metric_Pad1.15x1.40mm_HandSolder, symbol Device:C_Small
- added J1: USB_B_Micro, Connector_USB:USB_Micro-B_Molex_47346-0001, symbol Connector:USB_B_Micro
- added J10: Touch, Connector_PinHeader_2.54mm:PinHeader_1x04_P2.54mm_Vertical, symbol Connector_Generic:Conn_01x04
- added J2: Audio, Connector_PinSocket_2.54mm:PinSocket_1x04_P2.54mm_Vertical, symbol Connector_Generic:Conn_01x04
- added J6: UART, Connector_PinHeader_2.54mm:PinHeader_1x06_P2.54mm_Vertical, symbol Connector_Generic:Conn_01x06
- added J7: Micro_SD_Card, Connector_Card:microSD_HC_Wuerth_693072010801, symbol Connector:Micro_SD_Card
- added J8: LCD, Connector_PinHeader_2.54mm:PinHeader_1x06_P2.54mm_Vertical, symbol Connector_Generic:Conn_01x06
- added J9: Keypad, Connector_PinHeader_2.54mm:PinHeader_1x04_P2.54mm_Vertical, symbol Connector_Generic:Conn_01x04
- added R4, R5: 470, Resistor_SMD:R_0805_2012Metric_Pad1.15x1.40mm_HandSolder, symbol Device:R_US
- gave numbers to parts that had none: 1
Connections:
- net labels added: DAC, I2C_SCL, I2C_SDA, LCD_DC, PA0, PA1, PA2, PA3, PB8, PC12, SD_SPI_CLK, SD_SPI_CS, SD_SPI_MISO, SD_SPI_MOSI, SPI_CS, SPI_MOSI, SPI_SCK
- net labels removed: U5V, XPC14, XPC15, XPF0, XPF1
- wire segments 97 -> 188
- no-connect marks 1 -> 38
Other:
- moved on the sheet: C11, D1, LD1, R1, R10, R3, SW1

Commit message: added SD_SPI_MISO 10K pullup
Parts:
- removed D1: BAT60JFILM, Diode_SMD:D_SOD-323, symbol Diode:BAT60A
- added R6: 10K, Resistor_SMD:R_0805_2012Metric_Pad1.15x1.40mm_HandSolder, symbol Device:R_US
Connections:
- wire segments 188 -> 190
Changed lines of the file:
@@
 	1    0    0    -1
 $EndComp
-$Comp
-L Diode:BAT60A D1
-U 1 1 5EDEB2B3
-P 2350 1850
-F 0 "D1" H 2350 1633 50  0000 C CNN
-F 1 "BAT60JFILM" H 2350 1724 50  0000 C CNN
-F 2 "Diode_SMD:D_SOD-323" H 2350 1675 50  0001 C CNN
-F 3 "https://www.infineon.com/dgdl/Infineon-BAT60ASERIES-DS-v01_01-en.pdf?fileId=db3a304313d846880113def70c9304a9" H 2350 1850 50  0001 C CNN
-	1    2350 1850
-	-1   0    0    1
-$EndComp
-Wire Wire Line
-	2600 1850 2500 1850
 NoConn ~ 1650 2050
 NoConn ~ 1650 2150
@@
 	8100 1350 7550 1350
 Wire Wire Line
-	8100 1550 7550 1550
+	8100 1550 7700 1550
 Text Label 7550 1550 0    50   ~ 0
 SD_SPI_MISO
@@
 Wire Wire Line
 	5050 5900 5050 6000
-Wire Wire Line
-	1650 1850 2200 1850
 $Comp
 L power:PWR_FLAG #FLG0101
@@
 	1    0    0    -1
 $EndComp
+Wire Wire Line
+	1650 1850 2600 1850
+$Comp
+L Device:R_US R6
+U 1 1 61C2579F
+P 7700 1850
+F 0 "R6" H 7768 1896 50  0000 L CNN
+F 1 "10K" H 7768 1805 50  0000 L CNN
+F 2 "Resistor_SMD:R_0805_2012Metric_Pad1.15x1.40mm_HandSolder" V 7740 1840 50  0001 C CNN
+F 3 "" H 7700 1850 50  0001 C CNN
+	1    7700 1850
+	1    0    0    -1
+$EndComp
+$Comp
+L power:+3V0 #PWR01
+U 1 1 61C272C2
+P 7500 2000
+F 0 "#PWR01" H 7500 1850 50  0001 C CNN
+F 1 "+3V0" H 7515 2173 50  0000 C CNN
+F 2 "" H 7500 2000 50  0001 C CNN
+F 3 "" H 7500 2000 50  0001 C CNN
+	1    7500 2000
+	1    0    0    -1
+$EndComp
+Wire Wire Line
+	7500 2000 7700 2000
+Wire Wire Line
+	7700 1700 7700 1550
+Connection ~ 7700 1550
+Wire Wire Line
+	7700 1550 7550 1550
 $EndSCHEMATC
